Commit message: added support for Velodyne 16 and Velodyne HDL sensors

File: husky/husky_description/urdf/husky.urdf.xacro (robot description, xacro)
@@ -32,4 +32,6 @@
   <xacro:arg name="realsense_rpy" default="$(optenv HUSKY_REALSENSE_RPY 0 0 0)" />
   <xacro:arg name="realsense_mount" default="$(optenv HUSKY_REALSENSE_MOUNT_FRAME sensor_arch_mount_link)" />
+  <xacro:arg name="velodyne16_enabled" default="false" />
+  <xacro:arg name="velodyne32_enabled" default="false" />
   <xacro:property name="husky_front_bumper_extend" value="$(optenv HUSKY_FRONT_BUMPER_EXTEND 0)" />
   <xacro:property name="husky_rear_bumper_extend" value="$(optenv HUSKY_REAR_BUMPER_EXTEND 0)" />
@@ -129,4 +131,18 @@
     </joint>
   </xacro:if>
+  <!-- Add Velodyn-16 using Velodyn Simulator package -->
+  <xacro:if value="$(arg velodyne16_enabled)">
+    <xacro:include filename="$(find velodyne_description)/urdf/VLP-16.urdf.xacro"/>
+    <xacro:VLP-16 parent="base_link" name="velodyne" topic="/velodyne_points" hz="10" samples="440" gpu="false">
+      <origin xyz="0 0 0.45" rpy="0 0 0" />
+    </xacro:VLP-16>
+  </xacro:if>
+  <!-- Add Velodyn-16 using Velodyn Simulator package -->
+  <xacro:if value="$(arg velodyne32_enabled)">
+    <xacro:include filename="$(find velodyne_description)/urdf/HDL-32E.urdf.xacro"/>
+    <xacro:HDL-32E parent="base_link" name="velodyne2" topic="/velodyne_points2" hz="10" samples="220" gpu="false">
+      <origin xyz="0 0 0.6" rpy="0 0 0" />
+    </xacro:HDL-32E>
+  </xacro:if>
   <!-- top sensor arch; include this if we have either the kinect or realsense enabled -->
   <xacro:property name="topbar_needed_kinect" value="$(arg kinect_enabled)" />

Commit message: added support for velodyne 16

File: husky/husky_description/urdf/husky.urdf.xacro (robot description, xacro)
@@ -32,6 +32,5 @@
   <xacro:arg name="realsense_rpy" default="$(optenv HUSKY_REALSENSE_RPY 0 0 0)" />
   <xacro:arg name="realsense_mount" default="$(optenv HUSKY_REALSENSE_MOUNT_FRAME sensor_arch_mount_link)" />
-  <xacro:arg name="velodyne16_enabled" default="false" />
-  <xacro:arg name="velodyne32_enabled" default="false" />
+  <xacro:arg name="velodyne_enabled" default="false" />
   <xacro:property name="husky_front_bumper_extend" value="$(optenv HUSKY_FRONT_BUMPER_EXTEND 0)" />
   <xacro:property name="husky_rear_bumper_extend" value="$(optenv HUSKY_REAR_BUMPER_EXTEND 0)" />
@@ -132,16 +131,9 @@
   </xacro:if>
   <!-- Add Velodyn-16 using Velodyn Simulator package -->
-  <xacro:if value="$(arg velodyne16_enabled)">
+  <xacro:if value="$(arg velodyne_enabled)">
     <xacro:include filename="$(find velodyne_description)/urdf/VLP-16.urdf.xacro"/>
     <xacro:VLP-16 parent="base_link" name="velodyne" topic="/velodyne_points" hz="10" samples="440" gpu="false">
       <origin xyz="0 0 0.45" rpy="0 0 0" />
     </xacro:VLP-16>
-  </xacro:if>
-  <!-- Add Velodyn-16 using Velodyn Simulator package -->
-  <xacro:if value="$(arg velodyne32_enabled)">
-    <xacro:include filename="$(find velodyne_description)/urdf/HDL-32E.urdf.xacro"/>
-    <xacro:HDL-32E parent="base_link" name="velodyne2" topic="/velodyne_points2" hz="10" samples="220" gpu="false">
-      <origin xyz="0 0 0.6" rpy="0 0 0" />
-    </xacro:HDL-32E>
   </xacro:if>
   <!-- top sensor arch; include this if we have either the kinect or realsense enabled -->

Commit message: added kinetic packages for husky

File: husky/husky_description/urdf/husky.urdf.xacro (robot description, xacro)
@@ -25,12 +25,8 @@
   <xacro:arg name="laser_xyz" default="$(optenv HUSKY_LMS1XX_XYZ 0.2206 0.0 0.00635)" />
   <xacro:arg name="laser_rpy" default="$(optenv HUSKY_LMS1XX_RPY 0.0 0.0 0.0)" />
-  <xacro:arg name="kinect_enabled" default="false" />
-  <xacro:arg name="kinect_xyz" default="$(optenv HUSKY_KINECT_XYZ 0 0 0)" />
-  <xacro:arg name="kinect_rpy" default="$(optenv HUSKY_KINECT_RPY 0 0.18 3.14)" />
   <xacro:arg name="realsense_enabled" default="false" />
   <xacro:arg name="realsense_xyz" default="$(optenv HUSKY_REALSENSE_XYZ 0 0 0)" />
   <xacro:arg name="realsense_rpy" default="$(optenv HUSKY_REALSENSE_RPY 0 0 0)" />
   <xacro:arg name="realsense_mount" default="$(optenv HUSKY_REALSENSE_MOUNT_FRAME sensor_arch_mount_link)" />
-  <xacro:arg name="velodyne_enabled" default="false" />
   <xacro:property name="husky_front_bumper_extend" value="$(optenv HUSKY_FRONT_BUMPER_EXTEND 0)" />
   <xacro:property name="husky_rear_bumper_extend" value="$(optenv HUSKY_REAR_BUMPER_EXTEND 0)" />
@@ -40,5 +36,4 @@
   <xacro:include filename="$(find husky_description)/urdf/decorations.urdf.xacro" />
   <xacro:include filename="$(find husky_description)/urdf/wheel.urdf.xacro" />
-  <xacro:include filename="$(find husky_description)/urdf/accessories/kinect_camera.urdf.xacro"/>
   <xacro:include filename="$(find husky_description)/urdf/accessories/intel_realsense.urdf.xacro"/>
   <xacro:include filename="$(find husky_description)/urdf/accessories/sick_lms1xx_mount.urdf.xacro"/>
@@ -130,29 +125,11 @@
     </joint>
   </xacro:if>
-  <!-- Add Velodyn-16 using Velodyn Simulator package -->
-  <xacro:if value="$(arg velodyne_enabled)">
-    <xacro:include filename="$(find velodyne_description)/urdf/VLP-16.urdf.xacro"/>
-    <xacro:VLP-16 parent="base_link" name="velodyne" topic="/velodyne_points" hz="10" samples="440" gpu="false">
-      <origin xyz="0 0 0.45" rpy="0 0 0" />
-    </xacro:VLP-16>
-  </xacro:if>
-  <!-- top sensor arch; include this if we have either the kinect or realsense enabled -->
-  <xacro:property name="topbar_needed_kinect" value="$(arg kinect_enabled)" />
+  <!-- top sensor arch; include this if we have the realsense enabled -->
   <xacro:property name="topbar_needed_realsense" value="$(arg realsense_enabled)" />
   <!-- In melodic we can treat the above as booleans, but in kinetic they're strings, hence this ugliness... -->
-  <xacro:if value="${topbar_needed_kinect == 'true' or topbar_needed_kinect == '1' or topbar_needed_realsense == 'true' or topbar_needed_realsense == '1'}">
+  <xacro:if value="${topbar_needed_realsense == 'true' or topbar_needed_realsense == '1'}">
     <xacro:sensor_arch prefix="" parent="top_plate_link">
       <origin xyz="-0.35 0 0.51" rpy="0 0 -3.14"/>
     </xacro:sensor_arch>
-  </xacro:if>
-  <!-- add the kinect for xbox 360 to the topbar if needed -->
-  <!-- NOTE: this camera is considered depricated -->
-  <xacro:if value="$(arg kinect_enabled)">
-    <joint name="kinect_frame_joint" type="fixed">
-      <origin xyz="$(arg kinect_xyz)" rpy="$(arg kinect_rpy)" />
-      <parent link="sensor_arch_mount_link"/>
-      <child link="camera_link"/>
-    </joint>
-    <xacro:kinect_camera prefix="camera" robot_namespace="$(arg robot_namespace)"/>
   </xacro:if>
   <!-- add the intel realsense to the topbar if needed -->

Commit message: remove lms1XX

File: husky/husky_description/urdf/husky.urdf.xacro (robot description, xacro)
@@ -25,12 +25,8 @@
   <xacro:arg name="laser_xyz" default="$(optenv HUSKY_LMS1XX_XYZ 0.2206 0.0 0.00635)" />
   <xacro:arg name="laser_rpy" default="$(optenv HUSKY_LMS1XX_RPY 0.0 0.0 0.0)" />
-  <xacro:arg name="kinect_enabled" default="false" />
-  <xacro:arg name="kinect_xyz" default="$(optenv HUSKY_KINECT_XYZ 0 0 0)" />
-  <xacro:arg name="kinect_rpy" default="$(optenv HUSKY_KINECT_RPY 0 0.18 3.14)" />
   <xacro:arg name="realsense_enabled" default="false" />
   <xacro:arg name="realsense_xyz" default="$(optenv HUSKY_REALSENSE_XYZ 0 0 0)" />
   <xacro:arg name="realsense_rpy" default="$(optenv HUSKY_REALSENSE_RPY 0 0 0)" />
   <xacro:arg name="realsense_mount" default="$(optenv HUSKY_REALSENSE_MOUNT_FRAME sensor_arch_mount_link)" />
-  <xacro:arg name="velodyne_enabled" default="false" />
   <xacro:property name="husky_front_bumper_extend" value="$(optenv HUSKY_FRONT_BUMPER_EXTEND 0)" />
   <xacro:property name="husky_rear_bumper_extend" value="$(optenv HUSKY_REAR_BUMPER_EXTEND 0)" />
@@ -40,5 +36,4 @@
   <xacro:include filename="$(find husky_description)/urdf/decorations.urdf.xacro" />
   <xacro:include filename="$(find husky_description)/urdf/wheel.urdf.xacro" />
-  <xacro:include filename="$(find husky_description)/urdf/accessories/kinect_camera.urdf.xacro"/>
   <xacro:include filename="$(find husky_description)/urdf/accessories/intel_realsense.urdf.xacro"/>
   <xacro:include filename="$(find husky_description)/urdf/accessories/sick_lms1xx_mount.urdf.xacro"/>
@@ -84,5 +79,5 @@
     <child link="base_footprint" />
   </joint>
-  <!-- Interial link stores the robot's inertial information -->
+  <!-- Inertial link stores the robot's inertial information -->
   <link name="inertial_link">
     <inertial>
@@ -130,29 +125,14 @@
     </joint>
   </xacro:if>
-  <!-- Add Velodyn-16 using Velodyn Simulator package -->
-  <xacro:if value="$(arg velodyne_enabled)">
-    <xacro:include filename="$(find velodyne_description)/urdf/VLP-16.urdf.xacro"/>
-    <xacro:VLP-16 parent="base_link" name="velodyne" topic="/velodyne_points" hz="10" samples="440" gpu="false">
-      <origin xyz="0 0 0.45" rpy="0 0 0" />
-    </xacro:VLP-16>
-  </xacro:if>
-  <!-- top sensor arch; include this if we have either the kinect or realsense enabled -->
-  <xacro:property name="topbar_needed_kinect" value="$(arg kinect_enabled)" />
+  <!--
+    top sensor arch; include this if we have realsense enabled
+    keep this as a property to make it easier to add multiple conditions, should we need
+    the top bar for any additional sensors in the future
+  -->
   <xacro:property name="topbar_needed_realsense" value="$(arg realsense_enabled)" />
-  <!-- In melodic we can treat the above as booleans, but in kinetic they're strings, hence this ugliness... -->
-  <xacro:if value="${topbar_needed_kinect == 'true' or topbar_needed_kinect == '1' or topbar_needed_realsense == 'true' or topbar_needed_realsense == '1'}">
+  <xacro:if value="${topbar_needed_realsense}">
     <xacro:sensor_arch prefix="" parent="top_plate_link">
       <origin xyz="-0.35 0 0.51" rpy="0 0 -3.14"/>
     </xacro:sensor_arch>
-  </xacro:if>
-  <!-- add the kinect for xbox 360 to the topbar if needed -->
-  <!-- NOTE: this camera is considered depricated -->
-  <xacro:if value="$(arg kinect_enabled)">
-    <joint name="kinect_frame_joint" type="fixed">
-      <origin xyz="$(arg kinect_xyz)" rpy="$(arg kinect_rpy)" />
-      <parent link="sensor_arch_mount_link"/>
-      <child link="camera_link"/>
-    </joint>
-    <xacro:kinect_camera prefix="camera" robot_namespace="$(arg robot_namespace)"/>
   </xacro:if>
   <!-- add the intel realsense to the topbar if needed -->

Commit message: copy the stuff from original repo and modify laser joint stuff

File: husky/husky_description/urdf/husky.urdf.xacro (robot description, xacro)
@@ -29,4 +29,5 @@
   <xacro:arg name="realsense_rpy" default="$(optenv HUSKY_REALSENSE_RPY 0 0 0)" />
   <xacro:arg name="realsense_mount" default="$(optenv HUSKY_REALSENSE_MOUNT_FRAME sensor_arch_mount_link)" />
+  <xacro:arg name="velodyne_enabled" default="false" />
   <xacro:property name="husky_front_bumper_extend" value="$(optenv HUSKY_FRONT_BUMPER_EXTEND 0)" />
   <xacro:property name="husky_rear_bumper_extend" value="$(optenv HUSKY_REAR_BUMPER_EXTEND 0)" />
@@ -125,4 +126,11 @@
     </joint>
   </xacro:if>
+  <!-- Add Velodyn-16 using Velodyn Simulator package -->
+  <xacro:if value="$(arg velodyne_enabled)">
+    <xacro:include filename="$(find velodyne_description)/urdf/VLP-16.urdf.xacro"/>
+    <xacro:VLP-16 parent="base_link" name="velodyne" topic="/velodyne_points" hz="10" samples="440" gpu="false">
+      <origin xyz="0 0 0.45" rpy="0 0 0" />
+    </xacro:VLP-16>
+  </xacro:if>
   <!--
     top sensor arch; include this if we have realsense enabled

Commit message: added necessary packages for husky in noetic

File: husky/husky_description/urdf/husky.urdf.xacro (robot description, xacro)
@@ -25,12 +25,8 @@
   <xacro:arg name="laser_xyz" default="$(optenv HUSKY_LMS1XX_XYZ 0.2206 0.0 0.00635)" />
   <xacro:arg name="laser_rpy" default="$(optenv HUSKY_LMS1XX_RPY 0.0 0.0 0.0)" />
-  <xacro:arg name="kinect_enabled" default="false" />
-  <xacro:arg name="kinect_xyz" default="$(optenv HUSKY_KINECT_XYZ 0 0 0)" />
-  <xacro:arg name="kinect_rpy" default="$(optenv HUSKY_KINECT_RPY 0 0.18 3.14)" />
   <xacro:arg name="realsense_enabled" default="false" />
   <xacro:arg name="realsense_xyz" default="$(optenv HUSKY_REALSENSE_XYZ 0 0 0)" />
   <xacro:arg name="realsense_rpy" default="$(optenv HUSKY_REALSENSE_RPY 0 0 0)" />
   <xacro:arg name="realsense_mount" default="$(optenv HUSKY_REALSENSE_MOUNT_FRAME sensor_arch_mount_link)" />
-  <xacro:arg name="velodyne_enabled" default="false" />
   <xacro:property name="husky_front_bumper_extend" value="$(optenv HUSKY_FRONT_BUMPER_EXTEND 0)" />
   <xacro:property name="husky_rear_bumper_extend" value="$(optenv HUSKY_REAR_BUMPER_EXTEND 0)" />
@@ -40,5 +36,4 @@
   <xacro:include filename="$(find husky_description)/urdf/decorations.urdf.xacro" />
   <xacro:include filename="$(find husky_description)/urdf/wheel.urdf.xacro" />
-  <xacro:include filename="$(find husky_description)/urdf/accessories/kinect_camera.urdf.xacro"/>
   <xacro:include filename="$(find husky_description)/urdf/accessories/intel_realsense.urdf.xacro"/>
   <xacro:include filename="$(find husky_description)/urdf/accessories/sick_lms1xx_mount.urdf.xacro"/>
@@ -84,5 +79,5 @@
     <child link="base_footprint" />
   </joint>
-  <!-- Interial link stores the robot's inertial information -->
+  <!-- Inertial link stores the robot's inertial information -->
   <link name="inertial_link">
     <inertial>
@@ -122,6 +117,6 @@
   <xacro:husky_decorate />
   <xacro:if value="$(arg laser_enabled)">
-    <sick_lms1xx_mount prefix="base"/>
-    <sick_lms1xx frame="base_laser" topic="scan" robot_namespace="$(arg robot_namespace)"/>
+    <xacro:sick_lms1xx_mount prefix="base"/>
+    <xacro:sick_lms1xx frame="base_laser" topic="scan" robot_namespace="$(arg robot_namespace)"/>
     <joint name="laser_mount_joint" type="fixed">
       <origin xyz="$(arg laser_xyz)" rpy="$(arg laser_rpy)" />
@@ -130,29 +125,14 @@
     </joint>
   </xacro:if>
-  <!-- Add Velodyn-16 using Velodyn Simulator package -->
-  <xacro:if value="$(arg velodyne_enabled)">
-    <xacro:include filename="$(find velodyne_description)/urdf/VLP-16.urdf.xacro"/>
-    <xacro:VLP-16 parent="base_link" name="velodyne" topic="/velodyne_points" hz="10" samples="440" gpu="false">
-      <origin xyz="0 0 0.45" rpy="0 0 0" />
-    </xacro:VLP-16>
-  </xacro:if>
-  <!-- top sensor arch; include this if we have either the kinect or realsense enabled -->
-  <xacro:property name="topbar_needed_kinect" value="$(arg kinect_enabled)" />
+  <!--
+    top sensor arch; include this if we have realsense enabled
+    keep this as a property to make it easier to add multiple conditions, should we need
+    the top bar for any additional sensors in the future
+  -->
   <xacro:property name="topbar_needed_realsense" value="$(arg realsense_enabled)" />
-  <!-- In melodic we can treat the above as booleans, but in kinetic they're strings, hence this ugliness... -->
-  <xacro:if value="${topbar_needed_kinect == 'true' or topbar_needed_kinect == '1' or topbar_needed_realsense == 'true' or topbar_needed_realsense == '1'}">
+  <xacro:if value="${topbar_needed_realsense}">
     <xacro:sensor_arch prefix="" parent="top_plate_link">
       <origin xyz="-0.35 0 0.51" rpy="0 0 -3.14"/>
     </xacro:sensor_arch>
-  </xacro:if>
-  <!-- add the kinect for xbox 360 to the topbar if needed -->
-  <!-- NOTE: this camera is considered depricated -->
-  <xacro:if value="$(arg kinect_enabled)">
-    <joint name="kinect_frame_joint" type="fixed">
-      <origin xyz="$(arg kinect_xyz)" rpy="$(arg kinect_rpy)" />
-      <parent link="sensor_arch_mount_link"/>
-      <child link="camera_link"/>
-    </joint>
-    <xacro:kinect_camera prefix="camera" robot_namespace="$(arg robot_namespace)"/>
   </xacro:if>
   <!-- add the intel realsense to the topbar if needed -->
